File: WIFI-Relay_v0.2.sch (EAGLE design)
At the start: 38 parts, among them CN1 PBS-3-VERTICAL, CN2 PBS-2-VERTICAL, CN3 PBS-8-1.27-VERTICAL, CN4 PBS-8-1.27-VERTICAL, CN5 PBS-2-VERTICAL, CN6 PBS-2-VERTICAL, CN7 PBS-4-VERTICAL, IC1 74LS595D, IC2 74LS595D, IC3 MC34063AD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

Commit message: Value and name were changed. Eagle is 9.2.0
Parts:
- R10: value 5.1k -> 5.6k
